File: EDA files/EEZ DIB SMX46 r1B3.sch (EAGLE design)
At the start: 158 parts, among them IC1 STM32F030C6T6, IC2 74HC1G126GW,125, IC3 M24C32-WMN6P, IC4 LP2985-33DBVR, IC5 74HC2G04GW,125, IC6 OPA2990IDR, K1 FTR-C1GA012G-B05, K10 FTR-C1GA012G-B05, K11 FTR-C1GA012G-B05, K12 FTR-C1GA012G-B05, K13 FTR-C1GA012G-B05, K14 FTR-C1GA012G-B05, K15 FTR-C1GA012G-B05, K16 FTR-C1GA012G-B05, K17 FTR-C1GA012G-B05, K18 FTR-C1GA012G-B05, K19 FTR-C1GA012G-B05, K2 FTR-C1GA012G-B05, K20 FTR-C1GA012G-B05, K21 FTR-C1GA012G-B05, K22 FTR-C1GA012G-B05, K23 FTR-C1GA012G-B05, K24 FTR-C1GA012G-B05, K3 FTR-C1GA012G-B05, K4 FTR-C1GA012G-B05, K5 FTR-C1GA012G-B05, K6 FTR-C1GA012G-B05, K7 FTR-C1GA012G-B05, K8 FTR-C1GA012G-B05, K9 FTR-C1GA012G-B05, Q1 2N7002, Q10 2N7002, Q11 2N7002, Q12 2N7002, Q13 2N7002, Q14 2N7002, Q15 2N7002, Q16 2N7002, Q17 2N7002, Q18 2N7002, Q19 2N7002, Q2 2N7002, Q20 2N7002, Q21 2N7002, Q22 2N7002, Q23 2N7002, Q24 2N7002, Q25 2N7002, Q3 2N7002, Q4 2N7002, Q5 2N7002, Q6 2N7002, Q7 2N7002, Q8 2N7002, Q9 2N7002, X1 N.C., X2 77317-104-28LF, X3 691327310016, X4 691327310016

Commit message: #3
Connections:
- new net DIB_SYNC: IC1.PC15-OSC32_OUT, X2-6.1
Changed lines of the file:
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@@
 <setting verticaltext="up"/>
 </settings>
-<grid distance="0.1" unitdist="inch" unit="inch" style="lines" multiple="1" display="no" altdistance="0.01" altunitdist="inch" altunit="inch"/>
+<grid distance="0.025" unitdist="inch" unit="inch" style="lines" multiple="4" display="no" altdistance="0.01" altunitdist="inch" altunit="inch"/>
 <layers>
 <layer number="1" name="Top" color="4" fill="1" visible="no" active="no"/>
@@
 </segment>
 </net>
+<net name="DIB_SYNC" class="0">
+<segment>
+<pinref part="X2" gate="-6" pin="1"/>
+<wire x1="68.58" y1="152.4" x2="83.82" y2="152.4" width="0.1524" layer="91"/>
+<label x="83.82" y="153.035" size="1.27" layer="102" rot="MR0"/>
+</segment>
+<segment>
+<pinref part="IC1" gate="G$1" pin="PC15-OSC32_OUT"/>
+<wire x1="175.26" y1="111.76" x2="162.56" y2="111.76" width="0.1524" layer="91"/>
+<label x="162.56" y="112.395" size="1.27" layer="102"/>
+</segment>
+</net>
