File: EDA files/EEZ DIB SMX46 r1B4.brd (EAGLE design)
At the start: 146 x 95 mm, 159 parts, among them IC1 STM32F030C6T6, IC2 74HC1G126GW,125, IC3 M24C32-WMN6P, IC4 LP2985-33DBVR, IC5 74HC2G04GW,125, IC6 OPA2990IDR, K1 FTR-C1GA012G-B05, K10 FTR-C1GA012G-B05, K11 FTR-C1GA012G-B05, K12 FTR-C1GA012G-B05, K13 FTR-C1GA012G-B05, K14 FTR-C1GA012G-B05, K15 FTR-C1GA012G-B05, K16 FTR-C1GA012G-B05, K17 FTR-C1GA012G-B05, K18 FTR-C1GA012G-B05, K19 FTR-C1GA012G-B05, K2 FTR-C1GA012G-B05, K20 FTR-C1GA012G-B05, K21 FTR-C1GA012G-B05, K22 FTR-C1GA012G-B05, K23 FTR-C1GA012G-B05, K24 FTR-C1GA012G-B05, K3 FTR-C1GA012G-B05, K4 FTR-C1GA012G-B05, K5 FTR-C1GA012G-B05, K6 FTR-C1GA012G-B05, K7 FTR-C1GA012G-B05, K8 FTR-C1GA012G-B05, K9 FTR-C1GA012G-B05, Q1 2N7002, Q10 2N7002, Q11 2N7002, Q12 2N7002, Q13 2N7002, Q14 2N7002, Q15 2N7002, Q16 2N7002, Q17 2N7002, Q18 2N7002, Q19 2N7002, Q2 2N7002, Q20 2N7002, Q21 2N7002, Q22 2N7002, Q23 2N7002, Q24 2N7002, Q25 2N7002, Q3 2N7002, Q4 2N7002, Q5 2N7002, Q6 2N7002, Q7 2N7002, Q8 2N7002, Q9 2N7002, X1 N.C., X2 77317-104-28LF, X3 691327310016, X4 691327310016

Commit message: #4, OSHW UID
Parts:
- removed GND: (no value), EEZ_Lib1:PCB_SHIELD_TAB
- removed K_PWR: RT424005, EEZ_Lib1:RT-C/016A5_ROUND
- added FM3: FIDUCIAL_2, EEZ_Lib1:FIDUCIAL_DUAL
- added K25: FTR-C1GA012G-B05, EEZ_Lib1:FTR-C1
- added R15: 10K, rcl:R0805
- added TP1: (no value), EEZ_Lib1:PCB_SHIELD_TAB
- added U$3: HR000004, OSHWA:CERT-SMALL-SILK
- added X6, X7: DS1014-10RF1B, EEZ_connectors:DS1014-10RF1B
- C5: value 100n -> 2u2; device rcl:C0603 -> rcl:C0805
- C6: value 2u2 -> 100n; device rcl:C0805 -> rcl:C0603
- K19: value FTR-C1GA012G-B05 -> RT424005; device EEZ_Lib1:FTR-C1 -> EEZ_Lib1:RT-C/016A5_ROUND
- R10, R4: value 4K7 -> 10K
- R11, R5: value 10K -> 4K7
- R12, R6: value 47R -> 10K
- R13, R7: value 180R -> 47R
- R14, R8: value 10K -> 180R
- R2: value 47K -> 180R
- R3: value 10K -> 47K
- moved R12 33.0 mm to (98.2, 22.8), turned to 0 degrees
- moved R6 30.3 mm to (98.2, 27.4), turned to 0 degrees
- moved R14 27.8 mm to (75.1, 29.2)
- moved R9 27.1 mm to (102.1, 27.4)
- moved R3 26.2 mm to (61.4, 26.8), turned to 270 degrees
- moved R11 23.1 mm to (75.1, 23.3)
- moved K19 22.2 mm to (41.3, 21.1), turned to 180 degrees
- moved R7 19.7 mm to (67.9, 27.9), turned to 90 degrees
- moved K23 19.1 mm to (95.8, 41.3)
- moved K20 19.1 mm to (38.6, 41.3)
- moved K21 19.1 mm to (57.7, 41.3)
- moved K22 19.1 mm to (76.7, 41.3)
- moved K24 19.1 mm to (114.8, 41.3)
- moved R8 14.6 mm to (87.6, 29.2), turned to 0 degrees
- moved RN3 13.7 mm to (46.2, 81.8), turned to 0 degrees
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- renumbered DIB1.1 to JP1
Connections:
- net N$3 renamed Y3B
- net N$4 renamed Y3A
- removed net N$10: K19.5, K20.5, K21.5, K22.5, K23.5, K24.5, X3.16
- removed net N$11: K19.8, K20.8, K21.8, K22.8, K23.8, K24.8, X3.15
- removed net N$6: K10.5, K11.5, K12.5, K7.5, K8.5, K9.5, X3.12
- removed net N$7: K10.8, K11.8, K12.8, K7.8, K8.8, K9.8, X3.11
- removed net N$80: K1.5, K2.5, K3.5, K4.5, K5.5, K6.5, X3.10
- removed net N$81: K1.8, K2.8, K3.8, K4.8, K5.8, K6.8, X3.9
- new net N$77: Q1.1, R2.1, R3.2
- new net Y1A: K1.8, K2.8, K3.8, K4.8, K5.8, K6.8, X3.9, X6.4
- new net Y1B: K1.5, K2.5, K3.5, K4.5, K5.5, K6.5, X3.10, X6.3
- new net Y2A: K10.8, K11.8, K12.8, K7.8, K8.8, K9.8, X3.11, X7.4
- new net Y2B: K10.5, K11.5, K12.5, K7.5, K8.5, K9.5, X3.12, X7.3
- new net Y4A: K20.8, K21.8, K22.8, K23.8, K24.8, K25.8, X3.15
- new net Y4B: K20.5, K21.5, K22.5, K23.5, K24.5, K25.5, X3.16
- net +12V: now also K25.1; no longer K19.1
- net +3V3: now also C5.2, C6.1; no longer C5.1, C6.2
- net +5V: now also K19.A2; no longer K_PWR.A2
- net DAC#1: now also R6.1; no longer R5.1
- net DAC#2: now also R12.1; no longer R11.1
- net GND: now also C5.1, C6.2, R11.1, R3.1, R5.1, TP1.1; no longer C5.2, C6.1, GND.1, R10.1, R2.1, R4.1
- net ISET1: now also R7.1, R8.2; no longer R6.1, R7.2
- net ISET2: now also R13.1, R14.2; no longer R12.1, R13.2
- net K_PWR: no longer Q1.1
- net N$1: now also K20.4; no longer K19.4
- net N$100: now also K19.A1; no longer K_PWR.A1
- net N$12: now also K24.4; no longer K23.4
- net N$14: now also K21.4; no longer K20.4
- net N$15: now also K21.9; no longer K20.9
- net N$16: now also K24.9; no longer K23.9
- net N$17: now also K25.4; no longer K24.4
- net N$2: now also K20.9; no longer K19.9
- net N$20: now also K25.9; no longer K24.9
- net N$23: now also K21.12; no longer K20.12
- net N$24: now also K22.4; no longer K21.4
- net N$246: now also R9.1; no longer R8.1
- net N$25: now also K22.9; no longer K21.9
- net N$251: now also R4.1, R5.2; no longer R3.1, R4.2
- net N$252: now also R9.2; no longer R8.2
- net N$34: now also K23.4; no longer K22.4
- net N$35: now also K23.9; no longer K22.9
- net N$37: now also K22.12; no longer K21.12
- net N$47: now also K20.12; no longer K19.12
- net N$51: now also K23.12; no longer K22.12
- net N$57: now also K24.12; no longer K23.12
- net N$67: now also K25.12; no longer K24.12
- net N$68: now also R4.2, R7.2; no longer R3.2, R6.2
- net N$71: now also R15.1; no longer R14.1
- net N$73: now also R15.2; no longer R14.2
- net N$74: now also R8.1; no longer R7.1
- net N$76: now also R10.1, R11.2; no longer R10.2, R9.1
- net N$78: now also R14.1; no longer R13.1
- net N$82: now also K19.11B; no longer K_PWR.11B
- net N$84: now also K19.12B; no longer K_PWR.12B
- net N$86: now also R10.2, R13.2; no longer R12.2, R9.2
- net N$94: now also K19.14B; no longer K_PWR.14B
- net N$95: now also K19.11A; no longer K_PWR.11A
- net N$96: now also K19.12A; no longer K_PWR.12A
- net N$97: now also K19.14A; no longer K_PWR.14A
- net PWM#1: now also R6.2; no longer R5.2
- net PWM#2: now also R12.2; no longer R11.2
Routing:
- net Y2B: track 0.00 -> 175.6 mm, vias 0 -> 6
- net Y2A: track 0.00 -> 174.3 mm, vias 0 -> 7
- net Y1B: track 0.00 -> 167.6 mm, vias 0 -> 6
- net Y1A: track 0.00 -> 163.2 mm, vias 0 -> 6
- net Y4A: track 0.00 -> 158.1 mm, vias 0 -> 7
- net Y4B: track 0.00 -> 158.1 mm, vias 0 -> 7
- net N$11: track 156.2 -> 0.00 mm, vias 7 -> 0
- net N$10: track 156.2 -> 0.00 mm, vias 7 -> 0
- net N$80: track 153.2 -> 0.00 mm, vias 6 -> 0
- net N$6: track 152.8 -> 0.00 mm, vias 6 -> 0
- net N$81: track 151.9 -> 0.00 mm, vias 6 -> 0
- net N$7: track 151.4 -> 0.00 mm, vias 7 -> 0
- net +12V: track 732.5 -> 698.0 mm
- net OUT1: track 247.6 -> 224.3 mm, vias 4 -> 5
- net OUT0: track 237.6 -> 219.0 mm, vias 4 -> 5
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- added copper zone on layer 16, net N$3
Other:
- board text added: "+VAUX 2 NRESET 4 SYNC 6 SSDA 8 IRQ 10 CSB 12 MISO 14 GND 16 A2 18 GND 20 +12V 22 +5V 24 BOOT 26 UART_TX 28"
- board text added: "1 +3V3 3 NFAULT 5 SSCL 7 GND 9 CSA 11 GND 13 SCLK 15 MOSI 17 A0 19 A1 21 +12V 23 +5V 25 GND 27 UART_RX"
- board text added: "ADIB#1"
- board text added: "ADIB#2"
- board text added: "DIB (bottom view)"
- board text added: "EEZ DIB SMX46 (12/2020 r1B4)"
- board text added: "EEZ DIB SMX46 (12/2020 r1B4) Project source code: github.com/eez-open"
- board text removed: "EEZ DIB SMX46 (09/2020 r1B3)"
- board text removed: "EEZ DIB SMX46 (09/2020 r1B3) Project source code: github.com/eez-open"
