File: EDA files/EEZ DIB SMX46 r1B4.sch (EAGLE design)
At the start: 158 parts, among them IC1 STM32F030C6T6, IC2 74HC1G126GW,125, IC3 M24C32-WMN6P, IC4 LP2985-33DBVR, IC5 74HC2G04GW,125, IC6 OPA2990IDR, K1 FTR-C1GA012G-B05, K10 FTR-C1GA012G-B05, K11 FTR-C1GA012G-B05, K12 FTR-C1GA012G-B05, K13 FTR-C1GA012G-B05, K14 FTR-C1GA012G-B05, K15 FTR-C1GA012G-B05, K16 FTR-C1GA012G-B05, K17 FTR-C1GA012G-B05, K18 FTR-C1GA012G-B05, K19 FTR-C1GA012G-B05, K2 FTR-C1GA012G-B05, K20 FTR-C1GA012G-B05, K21 FTR-C1GA012G-B05, K22 FTR-C1GA012G-B05, K23 FTR-C1GA012G-B05, K24 FTR-C1GA012G-B05, K3 FTR-C1GA012G-B05, K4 FTR-C1GA012G-B05, K5 FTR-C1GA012G-B05, K6 FTR-C1GA012G-B05, K7 FTR-C1GA012G-B05, K8 FTR-C1GA012G-B05, K9 FTR-C1GA012G-B05, Q1 2N7002, Q10 2N7002, Q11 2N7002, Q12 2N7002, Q13 2N7002, Q14 2N7002, Q15 2N7002, Q16 2N7002, Q17 2N7002, Q18 2N7002, Q19 2N7002, Q2 2N7002, Q20 2N7002, Q21 2N7002, Q22 2N7002, Q23 2N7002, Q24 2N7002, Q25 2N7002, Q3 2N7002, Q4 2N7002, Q5 2N7002, Q6 2N7002, Q7 2N7002, Q8 2N7002, Q9 2N7002, X1 N.C., X2 77317-104-28LF, X3 691327310016, X4 691327310016

Commit message: #4, OSHW UID
Parts:
- removed K_PWR: RT424005, EEZ_Lib1:RELAY_RT314012-2
- added FM3: FIDUCIAL_2, EEZ_Lib1:FIDUCIAL_2
- added K25: FTR-C1GA012G-B05, EEZ_Lib1:FTR-C1
- added R15: 10K, rcl:R-EU_R0805
- added U$3: HR000004, OSHWA:CERT-SMALL
- added X6, X7: DS1014-10RF1B, EEZ_connectors:DS1014-10RF1B
- C5: value 100n -> 2u2; device rcl:C-EUC0603 -> rcl:C-EUC0805
- C6: value 2u2 -> 100n; device rcl:C-EUC0805 -> rcl:C-EUC0603
- K19: value FTR-C1GA012G-B05 -> RT424005; device EEZ_Lib1:FTR-C1 -> EEZ_Lib1:RELAY_RT314012-2
- R10, R4: value 4K7 -> 10K
- R11, R5: value 10K -> 4K7
- R12, R6: value 47R -> 10K
- R13, R7: value 180R -> 47R
- R14, R8: value 10K -> 180R
- R2: value 47K -> 180R
- R3: value 10K -> 47K
- renumbered DIB1.1 to JP1, GND to TP1
Connections:
- net N$3 renamed Y3B
- net N$4 renamed Y3A
- removed net N$10: K19-1.O, K20-1.O, K21-1.O, K22-1.O, K23-1.O, K24-1.O, X3-16.1
- removed net N$11: K19-2.O, K20-2.O, K21-2.O, K22-2.O, K23-2.O, K24-2.O, X3-15.1
- removed net N$6: K10-1.O, K11-1.O, K12-1.O, K7-1.O, K8-1.O, K9-1.O, X3-12.1
- removed net N$7: K10-2.O, K11-2.O, K12-2.O, K7-2.O, K8-2.O, K9-2.O, X3-11.1
- removed net N$80: K1-1.O, K2-1.O, K3-1.O, K4-1.O, K5-1.O, K6-1.O, X3-10.1
- removed net N$81: K1-2.O, K2-2.O, K3-2.O, K4-2.O, K5-2.O, K6-2.O, X3-9.1
- new net N$77: Q1.G, R2.1, R3.2
- new net Y1A: K1-2.O, K2-2.O, K3-2.O, K4-2.O, K5-2.O, K6-2.O, X3-9.1, X6-4.1
- new net Y1B: K1-1.O, K2-1.O, K3-1.O, K4-1.O, K5-1.O, K6-1.O, X3-10.1, X6-3.1
- new net Y2A: K10-2.O, K11-2.O, K12-2.O, K7-2.O, K8-2.O, K9-2.O, X3-11.1, X7-4.1
- new net Y2B: K10-1.O, K11-1.O, K12-1.O, K7-1.O, K8-1.O, K9-1.O, X3-12.1, X7-3.1
- new net Y4A: K20-2.O, K21-2.O, K22-2.O, K23-2.O, K24-2.O, K25-2.O, X3-15.1
- new net Y4B: K20-1.O, K21-1.O, K22-1.O, K23-1.O, K24-1.O, K25-1.O, X3-16.1
- net +12V: now also K25G$1.C1; no longer K19G$1.C1
- net +3V3: now also C5.2, C6.1; no longer C5.1, C6.2
- net +5V: now also K19K.C1; no longer K_PWRK.C1
- net DAC#1: now also R6.1; no longer R5.1
- net DAC#2: now also R12.1; no longer R11.1
- net GND: now also C5.1, C6.2, R11.1, R3.1, R5.1; no longer C5.2, C6.1, R10.1, R2.1, R4.1
- net ISET1: now also R7.1, R8.2; no longer R6.1, R7.2
- net ISET2: now also R13.1, R14.2; no longer R12.1, R13.2
- net K_PWR: no longer Q1.G
- net N$1: now also K20-1.P; no longer K19-1.P
- net N$100: now also K19K.C2; no longer K_PWRK.C2
- net N$12: now also K24-1.P; no longer K23-1.P
- net N$14: now also K21-1.P; no longer K20-1.P
- net N$15: now also K21-2.P; no longer K20-2.P
- net N$16: now also K24-2.P; no longer K23-2.P
- net N$17: now also K25-1.P; no longer K24-1.P
- net N$2: now also K20-2.P; no longer K19-2.P
- net N$20: now also K25-2.P; no longer K24-2.P
- net N$23: now also K21G$1.C2; no longer K20G$1.C2
- net N$24: now also K22-1.P; no longer K21-1.P
- net N$246: now also R9.1; no longer R8.1
- net N$25: now also K22-2.P; no longer K21-2.P
- net N$251: now also R4.1, R5.2; no longer R3.1, R4.2
- net N$252: now also R9.2; no longer R8.2
- net N$34: now also K23-1.P; no longer K22-1.P
- net N$35: now also K23-2.P; no longer K22-2.P
- net N$37: now also K22G$1.C2; no longer K21G$1.C2
- net N$47: now also K20G$1.C2; no longer K19G$1.C2
- net N$51: now also K23G$1.C2; no longer K22G$1.C2
- net N$57: now also K24G$1.C2; no longer K23G$1.C2
- net N$67: now also K25G$1.C2; no longer K24G$1.C2
- net N$68: now also R4.2, R7.2; no longer R3.2, R6.2
- net N$71: now also R15.1; no longer R14.1
- net N$73: now also R15.2; no longer R14.2
- net N$74: now also R8.1; no longer R7.1
- net N$76: now also R10.1, R11.2; no longer R10.2, R9.1
- net N$78: now also R14.1; no longer R13.1
- net N$82: now also K19-2.P; no longer K_PWR-2.P
- net N$84: now also K19-2.S; no longer K_PWR-2.S
- net N$86: now also R10.2, R13.2; no longer R12.2, R9.2
- net N$94: now also K19-2.O; no longer K_PWR-2.O
- net N$95: now also K19-1.P; no longer K_PWR-1.P
- net N$96: now also K19-1.S; no longer K_PWR-1.S
- net N$97: now also K19-1.O; no longer K_PWR-1.O
- net PWM#1: now also R6.2; no longer R5.2
- net PWM#2: now also R12.2; no longer R11.2
Other:
- note added: "ADIB connectors"
- moved on the sheet: C10, C5, C6, C7, C8, C9, D1, IC3, IC4, K19, K20, K21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
